File: hardware/Circut.kicad_pcb (KiCad board)
At the start: 2 copper layers, 28 parts, among them J1 USB_C_Receptacle_USB2.0_14P, J2 USB_B_Mini, J3 Jack-DC, J4 Conn_01x24_Pin, J5 Conn_01x24_Pin, J6 Conn_01x24_Pin, J7 Conn_01x03_Pin, U1 ESP32-WROOM-32, U2 AMS1117-3.3, U3 AMS1117CD-5.0, U4 INA219AxD, U5 INA219AxD

Commit message: Optimized backend and frontend
Parts:
- moved C1 227.1 mm to (140.2, 119.1)
- moved C2 227.1 mm to (123.2, 107.1)
- moved C3 227.1 mm to (134.2, 109.1)
- moved C4 227.1 mm to (126.8, 120.1)
- moved C5 227.1 mm to (141.8, 106.6)
- moved C6 227.1 mm to (120.8, 75.7)
- moved C7 227.1 mm to (164.2, 118.1)
- moved D1 227.1 mm to (128.7, 124.6)
- moved D2 227.1 mm to (140.2, 120.1)
- moved D3 227.1 mm to (121.8, 123.6)
- moved J2 227.1 mm to (144.8, 133.1)
- moved J3 227.1 mm to (117.8, 127.1)
- moved J4 227.1 mm to (155.9, 105.1)
- moved J5 227.1 mm to (164.6, 105.1)
- moved J6 227.1 mm to (173.4, 105.1)
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